File: pressure_sensor/_saved_pressure_sensor.sch (KiCad schematic (older format))
At the start: 14 parts, among them J1 SCREW_TERM, J2 SCREW_TERM, J3 S1, J4 S2, J5 S3, J6 S4, P1 SWD_TC, U1 STM32F042K4, U2 MS580314BA01-00, U3 MCP2551-I/SN

Commit message: finished pressure sensor board
Parts:
- U2: footprint MS580314BA01-00:XDCR_MS580314BA01-00 -> footprints:XDCR_MS580314BA01-00
Changed lines of the file:
@@
 F 0 "U2" H 9550 2450 50  0000 L CNN
 F 1 "MS580314BA01-00" H 9550 1050 50  0000 L CNN
-F 2 "MS580314BA01-00:XDCR_MS580314BA01-00" H 9950 1850 50  0001 L CNN
+F 2 "footprints:XDCR_MS580314BA01-00" H 9950 1850 50  0001 L CNN
 F 3 "17.19 USD" H 9950 1850 50  0001 L CNN
 F 4 "TE Connectivity" H 9950 1850 50  0001 L CNN "MF"
