File: pressure_sensor/pressure_sensor.sch (KiCad schematic (older format))
At the start: 14 parts, among them J1 SCREW_TERM, J2 SCREW_TERM, J3 S1, J4 S2, J5 S3, J6 S4, P1 SWD_TC, U1 STM32F042K4, U2 MS580314BA01-00, U3 MCP2551-I/SN

Commit message: finished pressure sensor
Parts:
- P1: footprint agg:TC2030-NL -> footprints:SWD_CONN
- U2: footprint MS580314BA01-00:XDCR_MS580314BA01-00 -> footprints:XDCR_MS580314BA01-00
Changed lines of the file:
@@
 F 0 "U2" H 9550 2450 50  0000 L CNN
 F 1 "MS580314BA01-00" H 9550 1050 50  0000 L CNN
-F 2 "MS580314BA01-00:XDCR_MS580314BA01-00" H 9950 1850 50  0001 L CNN
+F 2 "footprints:XDCR_MS580314BA01-00" H 9950 1850 50  0001 L CNN
 F 3 "17.19 USD" H 9950 1850 50  0001 L CNN
 F 4 "TE Connectivity" H 9950 1850 50  0001 L CNN "MF"
@@
 F 0 "P1" H 6550 4000 50  0000 L CNN
 F 1 "SWD_TC" H 6550 3600 50  0000 L CNN
-F 2 "agg:TC2030-NL" H 6550 3500 50  0001 L CNN
+F 2 "footprints:SWD_CONN" H 6550 3500 50  0001 L CNN
 F 3 "" H 6450 3900 50  0001 C CNN
 	1    6850 3800

Commit message: added STM shield
Parts:
- C1, C2: symbol CP -> CP-RESCUE-pressure_sensor
- R1, R2: symbol R -> R-RESCUE-pressure_sensor
Changed lines of the file:
@@
 EESchema Schematic File Version 2
-LIBS:power
-LIBS:device
-LIBS:transistors
-LIBS:conn
-LIBS:linear
-LIBS:regul
-LIBS:74xx
-LIBS:cmos4000
-LIBS:adc-dac
-LIBS:memory
-LIBS:xilinx
-LIBS:microcontrollers
-LIBS:dsp
-LIBS:microchip
-LIBS:analog_switches
-LIBS:motorola
-LIBS:texas
-LIBS:intel
-LIBS:audio
-LIBS:interface
-LIBS:digital-audio
-LIBS:philips
-LIBS:display
-LIBS:cypress
-LIBS:siliconi
-LIBS:opto
-LIBS:atmel
-LIBS:contrib
-LIBS:valves
+LIBS:pressure_sensor-rescue
+LIBS:cauv_lib
 LIBS:agg-kicad
-LIBS:cauv_lib
 LIBS:pressure_sensor-cache
 EELAYER 25 0
@@
 CANRXD
 $Comp
-L R R1
+L R-RESCUE-pressure_sensor R1
 U 1 1 58D2C257
 P 750 1200
@@
 $EndComp
 $Comp
-L R R2
+L R-RESCUE-pressure_sensor R2
 U 1 1 58D2C35C
 P 750 1900
@@
 $EndComp
 $Comp
-L CP C1
+L CP-RESCUE-pressure_sensor C1
 U 1 1 58D2C56A
 P 2400 5700
@@
 $EndComp
 $Comp
-L CP C2
+L CP-RESCUE-pressure_sensor C2
 U 1 1 58D2C828
 P 9900 1050
