File: motor_driver/motor_driver.sch (KiCad schematic (older format))
At the start: 16 parts, among them J1 MCU, J2 MOTOR1, J3 MOTOR2, J4 PVDD, J5 12V, U1 DRV8432DKD

Commit message: added STM shield
Parts:
- removed C5, C6, C7, C8: 100nF, agg:0805, symbol C
- removed J2: MOTOR1, agg:SIL-254P-02, symbol CONN_01x02
- removed J3: MOTOR2, agg:SIL-254P-02, symbol CONN_01x02
- removed J4: PVDD, agg:SIL-254P-02, symbol CONN_01x02
- removed J5: 12V, agg:SIL-254P-02, symbol CONN_01x02
- added C5: 100uF, symbol CP
- added J2: MOTOR2, symbol Screw_Terminal_1x02
- added J3: MOTOR1, symbol Screw_Terminal_1x02
- added J4: PVDD_CONN, symbol Screw_Terminal_1x02
- added J5: VDD_CONN, symbol Screw_Terminal_1x02
- C1, C2, C3, C4, C9: symbol C -> C-RESCUE-motor_driver
- R1: symbol R -> R-RESCUE-motor_driver
Connections:
- net labels added: PWM_A, PWM_B, PWM_C, PWM_D, RESET, VDD
- net labels removed: 12V
- wire segments 67 -> 71
Other:
- note added: "POWER SUPPLIES"
