File: STM32/STM32.sch (KiCad schematic (older format))
At the start: 7 parts, among them J1 Power_conn, P1 SWD_TC, U1 STM32F042K4, U2 LD1117S33TR, U3 STM32F042SHIELD

Commit message: finished protoying board
Parts:
- U3: footprint (none) -> footprints:STM32F042_SHIELD
Changed lines of the file:
@@
 F 0 "U3" H 5600 4250 60  0000 C CNN
 F 1 "STM32F042SHIELD" H 5750 2400 60  0000 C CNN
-F 2 "" V 5200 3100 60  0001 C CNN
+F 2 "footprints:STM32F042_SHIELD" V 5200 3100 60  0001 C CNN
 F 3 "" V 5200 3100 60  0001 C CNN
 	1    5600 3300
