File: light_board/light_board.kicad_pcb (KiCad board)
At the start: 2 copper layers, 36.2 x 33.7 mm, 17 parts, among them J1 CONN_01X02, J2 Screw_Terminal_1x02, J3 Screw_Terminal_1x02, Q1 FDC658AP, U1 LM3409MY

Commit message: checked the light board
Routing:
- added copper zone on F.Cu, net GND
Other:
- board size 36.2 x 33.7 mm -> 37.5 x 35 mm
- board text added: "GND"
- board text added: "LED+"
- board text added: "VDD"
